File: samples/MF2015/MF2015 Vertical.sch (EAGLE design)
At the start: 48 parts, among them IC1 LPC11U24FBD48/401, Q2 BC857B, Y2 12MHz

Commit message: Lots of work on layout and routing of the MF board.
Parts:
- removed U$1, U$2, U$3, U$4: FIDUCIAL, adafruit:FIDUCIAL
- removed Y2: 12MHz, microbuilder:CRYSTAL2.5X2.0MM
- added BAT1, BAT2: (no value), SparkFun-Electromechanical:BATTERYAAA-KIT
- added FID1, FID2, FID3, FID4: FIDUCIAL1X2, SparkFun-Aesthetics:FIDUCIAL1X2
- added IC2: LD117AS12TR, v-reg:LD117AS12TR
- added IC3: TPS61200, texas:TPS61200
- added Q1: (no value), JVN:CRYSTAL
- added R3: 1M, rcl:R-US_R0603
- R11, R2, R5: value 10k -> 10K
- R14: value 1.5k -> 1.5K
- R15: value 3k -> 3K
- R16: value 24k -> 24K
Connections:
- new net N$34: R3.2, U$5.ID
- new net N$37: BAT1.-, BAT2.+
- new net N$38: IC1.P1.31, L1.DIN
- net GND: now also BAT2.-, R3.1
- net N$25: now also Q1.2; no longer Y2.1
- net N$26: now also Q1.1; no longer Y2.2
Other:
- note removed: "USB_CONNECT"
- note removed: "USB_VBUS"
- moved on the sheet: R11, R2, S3, S4
